File: Audio.kicad_sch (KiCad schematic)
At the start: 15 parts, among them J5 AudioJack3_SwitchT, U2 MAX9850xTI

Commit message: Draft 2 Revision 2
Footprints still not all assigned.

Added: Test points, zero resistors, battery voltage monitor IC, PTC and zener surge protection on VBUS, UART connector

Changed: rerouted some signals, removed zener and resistor for reverse pol bat protection
Parts:
- added R47, R48, R49, R50, R51, R52: 0Ω, Resistor_SMD:R_0805_2012Metric, symbol Device:R_Small_US
Connections:
- net A_SDA is gone; now on net A_GPIO: R10.2, U2.28 (SDA)
- net A_SLC is gone; now on net A_GPIO: R11.2, U2.27 (SCL)
- net AGND: now also R47.2, R48.2, R49.2; no longer U2.10 (INL), U2.7 (ADD), U2.9 (INR)
- net A_GPIO: now also U2.9 (INR), R47.1
- net at U2.18 (HPR): now also R50.1; no longer J5.R
- net at U2.19 (HPL): now also R52.1; no longer J5.T
- net at U2.21 (HPS): now also R51.1; no longer J5.TN
- new net: R48.1, U2.10 (INL)
- new net: R49.1, U2.7 (ADD)
- new net: J5.R, R50.2
- new net: J5.T, R52.2
- new net: J5.TN, R51.2

Commit message: Remaining Footprint Added
Beware of footprints that come from online but do not match the kicad libraries - the pins might be mapped wrong!
Parts:
- J5: footprint Footprints:CLIFF_FC68131 -> Footprints:CUI_SJ-3524-SMT
Connections:
- net A_GPIO: no longer R10.2, R11.2, R47.1, U2.27 (SCL), U2.28 (SDA), U2.9 (INR)
- new net: R47.1, U2.9 (INR)
- new net A_SDA: R10.2, U2.28 (SDA)
- new net A_SLC: R11.2, U2.27 (SCL)
Other:
- note added: "Is the footprint for this guy event accessible? Who are we buyging from again?"
- note added: "THIS IC IS A TQFN chip! Be careful"
Changed lines of the file:
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@@
+		)
+	)
+	(text "Is the footprint for this guy event accessible? Who are\nwe buyging from again?"
+		(exclude_from_sim no)
+		(at 185.42 88.392 0)
+		(effects
+			(font
+				(size 1.27 1.27)
+				(color 255 23 0 1)
+			)
+		)
+	)
+	(text "THIS IC IS A TQFN chip! Be careful"
+		(exclude_from_sim no)
+		(at 140.208 64.008 0)
+		(effects
+			(font
+				(size 1.27 1.27)
+				(color 255 23 0 1)
+			)
 		)
 	)
@@
 	)
 	(junction
-		(at 99.06 88.9)
-		(diameter 0)
-		(color 0 0 0 0)
-	)
-	(junction
 		(at 45.72 69.85)
-		(diameter 0)
-		(color 0 0 0 0)
-	)
-	(junction
-		(at 99.06 99.06)
 		(diameter 0)
 		(color 0 0 0 0)
@@
 	)
 	(junction
-		(at 99.06 91.44)
-		(diameter 0)
-		(color 0 0 0 0)
-	)
-	(junction
 		(at 115.57 111.76)
 		(diameter 0)
@@
 	(wire
 		(pts
-			(xy 99.06 91.44) (xy 102.87 91.44)
+			(xy 87.63 91.44) (xy 102.87 91.44)
 		)
 		(stroke
@@
 	(wire
 		(pts
-			(xy 87.63 99.06) (xy 99.06 99.06)
+			(xy 87.63 99.06) (xy 102.87 99.06)
 		)
 		(stroke
@@
 	(wire
 		(pts
+			(xy 99.06 83.82) (xy 99.06 106.68)
+		)
+		(stroke
+			(width 0)
+			(type default)
+		)
+	)
+	(wire
+		(pts
 			(xy 99.06 116.84) (xy 101.6 116.84)
 		)
@@
 	(wire
 		(pts
-			(xy 99.06 88.9) (xy 99.06 91.44)
-		)
-		(stroke
-			(width 0)
-			(type default)
-		)
-	)
-	(wire
-		(pts
 			(xy 101.6 111.76) (xy 101.6 116.84)
 		)
@@
 	(wire
 		(pts
-			(xy 99.06 99.06) (xy 102.87 99.06)
-		)
-		(stroke
-			(width 0)
-			(type default)
-		)
-	)
-	(wire
-		(pts
-			(xy 99.06 99.06) (xy 99.06 106.68)
-		)
-		(stroke
-			(width 0)
-			(type default)
-		)
-	)
-	(wire
-		(pts
-			(xy 99.06 88.9) (xy 102.87 88.9)
+			(xy 87.63 88.9) (xy 102.87 88.9)
 		)
 		(stroke
@@
 	(wire
 		(pts
-			(xy 87.63 88.9) (xy 99.06 88.9)
-		)
-		(stroke
-			(width 0)
-			(type default)
-		)
-	)
-	(wire
-		(pts
 			(xy 118.11 111.76) (xy 118.11 119.38)
 		)
@@
 	(wire
 		(pts
-			(xy 99.06 91.44) (xy 99.06 99.06)
-		)
-		(stroke
-			(width 0)
-			(type default)
-		)
-	)
-	(wire
-		(pts
 			(xy 118.11 50.8) (xy 118.11 58.42)
 		)
@@
 	(wire
 		(pts
-			(xy 99.06 83.82) (xy 99.06 88.9)
-		)
-		(stroke
-			(width 0)
-			(type default)
-		)
-	)
-	(wire
-		(pts
 			(xy 90.17 71.12) (xy 102.87 71.12)
 		)
@@
 		(pts
 			(xy 152.4 91.44) (xy 154.94 91.44)
-		)
-		(stroke
-			(width 0)
-			(type default)
-		)
-	)
-	(wire
-		(pts
-			(xy 87.63 91.44) (xy 99.06 91.44)
 		)
 		(stroke
@@
 			)
 		)
-		(property "Footprint" "Footprints:CLIFF_FC68131"
+		(property "Footprint" "Footprints:CUI_SJ-3524-SMT"
 			(at 160.02 99.06 0)
 			(effects

Commit message: Components Placed on Layout
Added Power Management PMOS, Assigned missing footprints
Parts:
- added Q4: DMP3068L-7, Package_TO_SOT_SMD:SOT-23-3, symbol Simulation_SPICE:PMOS
- J5: value AudioJack3_SwitchT -> SJ-3524-SMT-TR
- TP1, TP2: footprint (none) -> TestPoint:TestPoint_Pad_1.5x1.5mm
Connections:
- net +3V3: now also Q4.3 (S); no longer C20.1, C21.1, C22.1, R10.1, R11.1, R12.1, U2.17 (AVDD), U2.26 (PVDD), U2.4 (DVDD)
- new net AVDD: C20.1, C21.1, C22.1, Q4.1 (D), R10.1, R11.1, R12.1, U2.17 (AVDD), U2.26 (PVDD), U2.4 (DVDD)
- new net PWR_CTRL: Q4.2 (G)

Commit message: Ratsnest organized
Certain pins on esp32 module changed to benefit layout. Named all decaps to dC. Current layout areas might be not optimal, i.e. complicated to wire
Parts:
- C29: footprint Capacitor_SMD:C_0805_2012Metric_Pad1.18x1.45mm_HandSolder -> Capacitor_SMD:C_0603_1608Metric_Pad1.08x0.95mm_HandSolder
- dC20: renamed from C20; footprint Capacitor_SMD:C_0805_2012Metric_Pad1.18x1.45mm_HandSolder -> Capacitor_SMD:C_0603_1608Metric_Pad1.08x0.95mm_HandSolder
- dC21: renamed from C21; footprint Capacitor_SMD:C_0805_2012Metric_Pad1.18x1.45mm_HandSolder -> Capacitor_SMD:C_0603_1608Metric_Pad1.08x0.95mm_HandSolder
- dC22: renamed from C22; footprint Capacitor_SMD:C_0805_2012Metric_Pad1.18x1.45mm_HandSolder -> Capacitor_SMD:C_0603_1608Metric_Pad1.08x0.95mm_HandSolder
- dC23: renamed from C23; footprint Capacitor_SMD:C_0805_2012Metric_Pad1.18x1.45mm_HandSolder -> Capacitor_SMD:C_0603_1608Metric_Pad1.08x0.95mm_HandSolder
- dC26: renamed from C26; footprint Capacitor_SMD:C_0805_2012Metric_Pad1.18x1.45mm_HandSolder -> Capacitor_SMD:C_0603_1608Metric_Pad1.08x0.95mm_HandSolder
- dC27: renamed from C27; footprint Capacitor_SMD:C_0805_2012Metric_Pad1.18x1.45mm_HandSolder -> Capacitor_SMD:C_0603_1608Metric_Pad1.08x0.95mm_HandSolder
- dC28: renamed from C28; footprint Capacitor_SMD:C_0805_2012Metric_Pad1.18x1.45mm_HandSolder -> Capacitor_SMD:C_0603_1608Metric_Pad1.08x0.95mm_HandSolder
Changed lines of the file:
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@@
 		(on_board yes)
 		(dnp no)
-		(property "Reference" "C22"
+		(property "Reference" "dC22"
 			(at 53.086 81.026 0)
 			(effects
@@
 			)
 		)
-		(property "Footprint" "Capacitor_SMD:C_0805_2012Metric_Pad1.18x1.45mm_HandSolder"
+		(property "Footprint" "Capacitor_SMD:C_0603_1608Metric_Pad1.08x0.95mm_HandSolder"
 			(at 52.07 78.74 0)
 			(effects
@@
 			(project "Media Player"
 				(path "/5c19345b-3707-4c90-b593-78a9c3e56866/31bc7b2c-ab8b-4c9e-a1df-dec3026ddee0"
-					(reference "C22")
+					(reference "dC22")
 					(unit 1)
 				)
@@
 		(on_board yes)
 		(dnp no)
-		(property "Reference" "C21"
+		(property "Reference" "dC21"
 			(at 59.944 81.026 0)
 			(effects
@@
 			)
 		)
-		(property "Footprint" "Capacitor_SMD:C_0805_2012Metric_Pad1.18x1.45mm_HandSolder"
+		(property "Footprint" "Capacitor_SMD:C_0603_1608Metric_Pad1.08x0.95mm_HandSolder"
 			(at 58.42 78.74 0)
 			(effects
@@
 			(project "Media Player"
 				(path "/5c19345b-3707-4c90-b593-78a9c3e56866/31bc7b2c-ab8b-4c9e-a1df-dec3026ddee0"
-					(reference "C21")
+					(reference "dC21")
 					(unit 1)
 				)
@@
 		(on_board yes)
 		(dnp no)
-		(property "Reference" "C28"
+		(property "Reference" "dC28"
 			(at 124.714 115.824 0)
 			(effects
@@
 			)
 		)
-		(property "Footprint" "Capacitor_SMD:C_0805_2012Metric_Pad1.18x1.45mm_HandSolder"
+		(property "Footprint" "Capacitor_SMD:C_0603_1608Metric_Pad1.08x0.95mm_HandSolder"
 			(at 121.92 116.84 0)
 			(effects
@@
 			(project "Media Player"
 				(path "/5c19345b-3707-4c90-b593-78a9c3e56866/31bc7b2c-ab8b-4c9e-a1df-dec3026ddee0"
-					(reference "C28")
+					(reference "dC28")
 					(unit 1)
 				)
@@
 		(on_board yes)
 		(dnp no)
-		(property "Reference" "C23"
+		(property "Reference" "dC23"
 			(at 168.402 66.802 0)
 			(effects
@@
 			)
 		)
-		(property "Footprint" "Capacitor_SMD:C_0805_2012Metric_Pad1.18x1.45mm_HandSolder"
+		(property "Footprint" "Capacitor_SMD:C_0603_1608Metric_Pad1.08x0.95mm_HandSolder"
 			(at 167.64 64.77 0)
 			(effects
@@
 			(project "Media Player"
 				(path "/5c19345b-3707-4c90-b593-78a9c3e56866/31bc7b2c-ab8b-4c9e-a1df-dec3026ddee0"
-					(reference "C23")
+					(reference "dC23")
 					(unit 1)
 				)
@@
 			)
 		)
-		(property "Footprint" "Capacitor_SMD:C_0805_2012Metric_Pad1.18x1.45mm_HandSolder"
+		(property "Footprint" "Capacitor_SMD:C_0603_1608Metric_Pad1.08x0.95mm_HandSolder"
 			(at 140.97 87.63 0)
 			(effects
@@
 		(on_board yes)
 		(dnp no)
-		(property "Reference" "C20"
+		(property "Reference" "dC20"
 			(at 66.802 80.772 0)
 			(effects
@@
 			)
 		)
-		(property "Footprint" "Capacitor_SMD:C_0805_2012Metric_Pad1.18x1.45mm_HandSolder"
+		(property "Footprint" "Capacitor_SMD:C_0603_1608Metric_Pad1.08x0.95mm_HandSolder"
 			(at 66.04 78.74 0)
 			(effects
@@
 			(project ""
 				(path "/5c19345b-3707-4c90-b593-78a9c3e56866/31bc7b2c-ab8b-4c9e-a1df-dec3026ddee0"
-					(reference "C20")
+					(reference "dC20")
 					(unit 1)
 				)
@@
 		(on_board yes)
 		(dnp no)
-		(property "Reference" "C27"
+		(property "Reference" "dC27"
 			(at 183.642 66.802 0)
 			(effects
@@
 			)
 		)
-		(property "Footprint" "Capacitor_SMD:C_0805_2012Metric_Pad1.18x1.45mm_HandSolder"
+		(property "Footprint" "Capacitor_SMD:C_0603_1608Metric_Pad1.08x0.95mm_HandSolder"
 			(at 182.88 64.77 0)
 			(effects
@@
 			(project "Media Player"
 				(path "/5c19345b-3707-4c90-b593-78a9c3e56866/31bc7b2c-ab8b-4c9e-a1df-dec3026ddee0"
-					(reference "C27")
+					(reference "dC27")
 					(unit 1)
 				)
@@
 		(on_board yes)
 		(dnp no)
-		(property "Reference" "C26"
+		(property "Reference" "dC26"
 			(at 176.022 66.802 0)
 			(effects
@@
 			)
 		)
-		(property "Footprint" "Capacitor_SMD:C_0805_2012Metric_Pad1.18x1.45mm_HandSolder"
+		(property "Footprint" "Capacitor_SMD:C_0603_1608Metric_Pad1.08x0.95mm_HandSolder"
 			(at 175.26 64.77 0)
 			(effects
@@
 			(project "Media Player"
 				(path "/5c19345b-3707-4c90-b593-78a9c3e56866/31bc7b2c-ab8b-4c9e-a1df-dec3026ddee0"
-					(reference "C26")
-					(unit 1)
-				)
+					(reference "dC26")
+					(unit 1)
+				)

Commit message: Added alternative audio IC
Added a SOP package audio IC (for easier board bring up) in hopes to replace MAX9850. Pins not fully mapped yet.
Other:
- moved on the sheet: C29, J5, Q4, R10, R11, R12, R47, R48, R49, R50, R51, R52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
