File: _autosave-Media Player.kicad_sch (KiCad schematic)
At the start: 73 parts, among them J1 12402012E212A, J10 MEM2075-00-140-01-A, J40 PH2.0, J41 UART, Q10 DMP3068L-7, Q40 DMP3068L-7, SW30 BOOT, SW31 RESET, SW32 SW_Push, SW33 SW_Push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

Commit message: Minor Changes
Power traces enlarged, certain pad and hole clearances on USB modified, still within design rules, fixed silk screen clearance, copper pours now with thermal relief for pads connected to large planes. Most DRC's resolved. Design rule constraints tuned very slightly.
Parts:
- TP3, TP4, TP5, TP6, TP7, TP8: footprint TestPoint:TestPoint_Pad_1.5x1.5mm -> footprints:TestPoint_Pad_1.5x1.5mm
Changed lines of the file:
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@@
 			)
 		)
-		(property "Footprint" "TestPoint:TestPoint_Pad_1.5x1.5mm"
+		(property "Footprint" "footprints:TestPoint_Pad_1.5x1.5mm"
 			(at 166.37 74.93 0)
 			(effects
@@
 			)
 		)
-		(property "Footprint" "TestPoint:TestPoint_Pad_1.5x1.5mm"
+		(property "Footprint" "footprints:TestPoint_Pad_1.5x1.5mm"
 			(at 166.37 77.47 0)
 			(effects
@@
 			)
 		)
-		(property "Footprint" "TestPoint:TestPoint_Pad_1.5x1.5mm"
+		(property "Footprint" "footprints:TestPoint_Pad_1.5x1.5mm"
 			(at 166.37 57.15 0)
 			(effects
@@
 			)
 		)
-		(property "Footprint" "TestPoint:TestPoint_Pad_1.5x1.5mm"
+		(property "Footprint" "footprints:TestPoint_Pad_1.5x1.5mm"
 			(at 135.89 39.37 0)
 			(effects
@@
 			)
 		)
-		(property "Footprint" "TestPoint:TestPoint_Pad_1.5x1.5mm"
+		(property "Footprint" "footprints:TestPoint_Pad_1.5x1.5mm"
 			(at 166.37 59.69 0)
 			(effects
@@
 			)
 		)
-		(property "Footprint" "TestPoint:TestPoint_Pad_1.5x1.5mm"
+		(property "Footprint" "footprints:TestPoint_Pad_1.5x1.5mm"
 			(at 166.37 54.61 0)
 			(effects
