File: AudioAlt.kicad_sch (KiCad schematic)
At the start: 36 parts, among them J70 PJ-327C-4A, Q70 DMP3068L-7, U70 WM8731SEDS

Commit message: No changes made.
Parts:
- J70: value PJ-327C-4A -> PJ-327A
Changed lines of the file:
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@@
 			)
 		)
-		(property "Value" "PJ-327C-4A"
+		(property "Value" "PJ-327A"
 			(at 256.54 98.4249 0)
 			(effects
@@
 			)
 		)
-		(property "Datasheet" "https://www.lcsc.com/product-detail/C145813.html?s_z=n_SJ-2524-SMT-TR"
+		(property "Datasheet" "https://www.lcsc.com/datasheet/C49284723.pdf"
 			(at 248.92 100.33 0)
 			(effects

Commit message: ORDERED: Updated Footprints, Silk Screen, Mounting Holes
Minor changes. This is the version sent to JLC
Parts:
- removed R81: 47kΩ, Resistor_SMD:R_0603_1608Metric_Pad0.98x0.95mm_HandSolder, symbol Device:R_Small_US
- added R95: 10kΩ, Resistor_SMD:R_0603_1608Metric_Pad0.98x0.95mm_HandSolder, symbol Device:R_Small_US
- added TP74: BIAS, footprints:TestPoint_Pad_1.5x1.5mm, symbol Connector:TestPoint
Connections:
- net A2_TSW: now also R95.2
- net AVDD: now also R95.1
- net at U70.17 (MICBIAS): now also TP74.1
Changed lines of the file:
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@@
 	)
 	(junction
-		(at 185.42 118.11)
-		(diameter 0)
-		(color 0 0 0 0)
-	)
-	(junction
 		(at 132.08 95.25)
 		(diameter 0)
@@
 	(wire
 		(pts
-			(xy 177.8 118.11) (xy 171.45 118.11)
-		)
-		(stroke
-			(width 0)
-			(type default)
-		)
-	)
-	(wire
-		(pts
 			(xy 116.84 105.41) (xy 124.46 105.41)
 		)
@@
 	(wire
 		(pts
-			(xy 182.88 118.11) (xy 185.42 118.11)
-		)
-		(stroke
-			(width 0)
-			(type default)
-		)
-	)
-	(wire
-		(pts
 			(xy 83.82 114.3) (xy 135.89 114.3)
 		)
@@
 	(wire
 		(pts
+			(xy 240.03 85.09) (xy 242.57 85.09)
+		)
+		(stroke
+			(width 0)
+			(type default)
+		)
+	)
+	(wire
+		(pts
 			(xy 148.59 71.12) (xy 148.59 63.5)
 		)
@@
 	(wire
 		(pts
+			(xy 229.87 85.09) (xy 234.95 85.09)
+		)
+		(stroke
+			(width 0)
+			(type default)
+		)
+	)
+	(wire
+		(pts
 			(xy 90.17 55.88) (xy 90.17 48.26)
 		)
@@
 	(wire
 		(pts
-			(xy 185.42 118.11) (xy 185.42 123.19)
+			(xy 185.42 113.03) (xy 185.42 123.19)
 		)
 		(stroke
@@
 	(wire
 		(pts
-			(xy 185.42 113.03) (xy 185.42 118.11)
-		)
-		(stroke
-			(width 0)
-			(type default)
-		)
-	)
-	(wire
-		(pts
 			(xy 124.46 105.41) (xy 132.08 105.41)
 		)
@@
 		)
 	)
+	(label "AVDD"
+		(at 229.87 85.09 180)
+		(effects
+			(font
+				(size 1.27 1.27)
+			)
+			(justify right bottom)
+		)
+	)
 	(label "HPVDD"
 		(at 158.75 63.5 270)
@@
 	(symbol
 		(lib_id "Device:R_Small_US")
-		(at 180.34 118.11 270)
+		(at 250.19 85.09 90)
+		(mirror x)
 		(unit 1)
 		(exclude_from_sim no)
@@
 		(on_board yes)
 		(dnp no)
-		(property "Reference" "R81"
-			(at 186.436 117.856 90)
+		(property "Reference" "R85"
+			(at 248.031 80.391 90)
 			(effects
 				(font
 					(size 1.27 1.27)
 				)
-				(justify left)
+				(justify right)
 			)
 		)
-		(property "Value" "47kΩ"
-			(at 191.77 117.856 90)
+		(property "Value" "10kΩ"
+			(at 248.158 82.042 90)
 			(effects
 				(font
 					(size 1.27 1.27)
 				)
-				(justify left)
+				(justify right)
 			)
 		)
 		(property "Footprint" "Resistor_SMD:R_0603_1608Metric_Pad0.98x0.95mm_HandSolder"
-			(at 180.34 118.11 0)
+			(at 250.19 85.09 0)
 			(effects
 				(font
@@
 		)
 		(property "Datasheet" "~"
-			(at 180.34 118.11 0)
+			(at 250.19 85.09 0)
 			(effects
 				(font
@@
 		)
 		(property "Description" "Resistor, small US symbol"
-			(at 180.34 118.11 0)
+			(at 250.19 85.09 0)
 			(effects
 				(font
@@
 			(project "Media Player"
 				(path "/5c19345b-3707-4c90-b593-78a9c3e56866/f44db6d7-c45e-4150-a777-8c6c189bba1b"
-					(reference "R81")
+					(reference "R85")
 					(unit 1)
 				)
@@
 	(symbol
 		(lib_id "Device:R_Small_US")
-		(at 250.19 85.09 90)
+		(at 237.49 85.09 90)
 		(mirror x)
 		(unit 1)
@@
 		(on_board yes)
 		(dnp no)
-		(property "Reference" "R85"
-			(at 249.428 78.994 0)
+		(property "Reference" "R95"
+			(at 235.966 80.772 90)
 			(effects
 				(font
 					(size 1.27 1.27)
 				)
-				(justify left)
+				(justify right)
 			)
 		)
 		(property "Value" "10kΩ"
-			(at 251.206 77.47 0)
+			(at 235.966 82.55 90)
 			(effects
 				(font
 					(size 1.27 1.27)
 				)
-				(justify left)
+				(justify right)
 			)
 		)
 		(property "Footprint" "Resistor_SMD:R_0603_1608Metric_Pad0.98x0.95mm_HandSolder"
-			(at 250.19 85.09 0)
+			(at 237.49 85.09 0)
 			(effects
 				(font
@@
 		)
 		(property "Datasheet" "~"
-			(at 250.19 85.09 0)
+			(at 237.49 85.09 0)
 			(effects
 				(font
@@
 		)
 		(property "Description" "Resistor, small US symbol"
-			(at 250.19 85.09 0)
+			(at 237.49 85.09 0)
 			(effects
 				(font
@@
 			(project "Media Player"
 				(path "/5c19345b-3707-4c90-b593-78a9c3e56866/f44db6d7-c45e-4150-a777-8c6c189bba1b"
-					(reference "R85")
+					(reference "R95")
 					(unit 1)
 				)
@@
 					(unit 1)
 				)
+			)
+		)
+	)
+	(symbol
+		(lib_id "Connector:TestPoint")
+		(at 171.45 118.11 270)
+		(unit 1)
+		(exclude_from_sim no)
+		(in_bom yes)
+		(on_board yes)
+		(dnp no)
+		(property "Reference" "TP74"
+			(at 176.53 116.8399 90)
+			(effects
+				(font
+					(size 1.27 1.27)
+				)
+				(justify left)
+			)
+		)
+		(property "Value" "BIAS"
+			(at 176.53 118.872 90)
+			(effects
+				(font
+					(size 1.27 1.27)
+				)
+				(justify left)
+			)
+		)
+		(property "Footprint" "footprints:TestPoint_Pad_1.5x1.5mm"
+			(at 171.45 123.19 0)
+			(effects
+				(font
+					(size 1.27 1.27)
+				)
+				(hide yes)
+			)
+		)
+		(property "Datasheet" "~"
+			(at 171.45 123.19 0)
+			(effects
+				(font
+					(size 1.27 1.27)
+				)
+				(hide yes)
+			)
+		)
+		(property "Description" "test point"
+			(at 171.45 118.11 0)
+			(effects
+				(font
+					(size 1.27 1.27)
+				)
+				(hide yes)
+			)
+		)
+		(pin "1"
+		)
+		(instances
+			(project "Media Player"
+				(path "/5c19345b-3707-4c90-b593-78a9c3e56866/f44db6d7-c45e-4150-a777-8c6c189bba1b"
+					(reference "TP74")
+					(unit 1)
+				)
